File: PCB/HackPad.kicad_pcb (KiCad board)
At the start: 2 copper layers, 65 x 83 mm, 25 parts, among them SW1 SW_Push, SW2 SW_Push, SW3 SW_Push, SW4 SW_Push, SW5 SW_Push, SW6 SW_Push, SW7 SW_Push, SW8 SW_Push, SW9 SW_Push, U1 XIAO-RP2040-DIP

Commit message: Add files via upload
Parts:
- added GND: TestPoint, TestPoint:TestPoint_Pad_D2.0mm, F.Cu at (80.1, 60.0)
- added GND: TestPoint, TestPoint:TestPoint_Pad_D2.0mm, F.Cu at (99.0, 67.5)
- added LED: TestPoint, TestPoint:TestPoint_Pad_D2.0mm, F.Cu at (95.0, 67.5)
- added LED: LED, TestPoint:TestPoint_Pad_D2.0mm, F.Cu at (84.6, 60.0)
- added VCC: TestPoint, TestPoint:TestPoint_Pad_D2.0mm, F.Cu at (103.0, 67.5)
- added VCC: TestPoint, TestPoint:TestPoint_Pad_D2.0mm, F.Cu at (75.7, 60.0)
- moved D11 22.3 mm to (83.3, 60.0)
- moved D10 22.0 mm to (76.9, 60.0)
- moved VCC 12.0 mm to (116.5, 67.5)
- moved SCL 8.00 mm to (128.5, 67.5)
- moved SDL 8.00 mm to (124.5, 67.5)
- moved VSS 4.00 mm to (120.5, 67.5)
- renumbered SCL1 to SCL, SDL1 to SDL, VCC1 to VCC, VSS1 to VSS
Routing:
- net Net-(D10-DIN): track 11.7 -> 40.1 mm, vias 0 -> 1
- net GND: track 53.6 -> 67.1 mm, vias 0 -> 1
- net Net-(U1-GPIO3/MOSI): track 43.5 -> 51.5 mm
- net Net-(U1-GPIO4/MISO): track 36.4 -> 44.2 mm
- net +5V: track 60.7 -> 65.6 mm, vias 0 -> 1
- net Net-(D10-DOUT): track 3.96 -> 7.23 mm
Other:
- board size 65 x 83 mm -> 65 x 90 mm
